File: FrontPanel.sch (KiCad schematic (older format))
At the start: 0 parts

Commit message: Adds Beam Modulation PCB
Changed lines of the file:
@@
 $Descr A4 11693 8268
 encoding utf-8
-Sheet 12 18
+Sheet 12 19
 Title ""
 Date ""
@@
 Text HLabel 9550 3650 2    60   Input ~ 0
 ElectronOptics
+Text HLabel 9550 3900 2    60   Input ~ 0
+BeamModulation
 $EndSCHEMATC
